Commit message: gazebo hand of god plugin

File: agni_description/robots/shadow_hand.urdf.xacro (robot description, xacro)
@@ -35,3 +35,13 @@
     <xacro:shadow_gazebo_controller_manager namespace="${prefix}" />
   </xacro:macro>
+  <!--       <gazebo>
+  <plugin name="hand_of_god" filename="libgazebo_ros_hand_of_god.so">
+    <robotNamespace></robotNamespace>
+    <linkName>r_shadow_motor_right::rh_forearm</linkName>
+    <frameId>hand</frameId>
+    <kl>200</kl>
+    <ka>200</ka>
+  </plugin>
+    </gazebo>
+ -->
 </robot>

File: agni_description/robots/single.urdf.xacro (robot description, xacro)
@@ -36,3 +36,14 @@
 	<xacro:arm_with_tool parent="${parent}" arm_type="$(arg ARM)" tool_type="$(arg TOOL)"
 	                     prefix="${PREFIX if PREFIX not in ['', '-'] else ''}"/>
+	<xacro:property name="PLUGIN_HAND" value="hand_$(arg PREFIX)"/>
+ 	<xacro:property name="LINK_NAME" value="$(arg PREFIX)_$(arg TOOL)::$(arg PREFIX)h_forearm"/>
+	<gazebo>
+		<plugin name="hand_of_god" filename="libgazebo_ros_hand_of_god.so">
+		<robotNamespace></robotNamespace>
+		<linkName>${LINK_NAME}</linkName>
+		<frameId>${PLUGIN_HAND}</frameId>
+		<kl>200</kl>
+		<ka>200</ka>
+		</plugin>
+	</gazebo>
 </robot>
